File: X-B350W-4-LITE-350W-CLASS-B-POWER-AMP-MAIN-CIRCUIT.kicad_sch (KiCad schematic)
At the start: 109 parts, among them Q4001 2N5401, Q4002 2N5401, Q4003 2N5401, Q4004 2N5551, Q4005 2N5551, Q4006 2N5551, Q4007 2N5551, Q4008 2N5401, Q4009 2N5551, Q4010 2N5551, Q4011 MJE15034G, Q4012 MJE15035G, Q4013 2SC5200, Q4014 2SC5200, Q4015 2SC5200, Q4016 2SA1943, Q4017 2SA1943, Q4018 2SA1943

Commit message: Update
Other:
- note added: ".title X-B350W-4-LITE SIMPLIFIED 350W CLASS-B POWER AMPLIFIER MAIN-CIRCUIT FOR 4-OHMS OUTPUT LOAD"
- note removed: ".title 350W CLASS-B POWER AMPLIFIER MAIN-CIRCUIT FOR 4-OHMS OUTPUT LOAD"
Changed lines of the file:
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@@
 		)
 	)
-	(text ".title 350W CLASS-B POWER AMPLIFIER MAIN-CIRCUIT FOR 4-OHMS OUTPUT LOAD"
+	(text ".title X-B350W-4-LITE SIMPLIFIED 350W CLASS-B POWER AMPLIFIER MAIN-CIRCUIT FOR 4-OHMS OUTPUT LOAD"
 		(exclude_from_sim no)
 		(at -184.15 89.535 0)
